File: Hardware/wardrobe_closer.sch (EAGLE design)
At the start: 9 parts, among them U1 ATTINY25-20SHR

Commit message: Update design
Parts:
- removed SENS-1: TCRT5000, qfm-trx1-24g:TCRT5000
- removed SG1: F/QMBIII, buzzer:F/QMBIII
- added D1, D2: WP7113SGD, LED:WP7113SGD
- added Q1: EVERLIGHT_PT334-6BEVERLIGHT_PT334-6B_0_0, Everlight - PT334-6B:EVERLIGHT_PT334-6BEVERLIGHT_PT334-6B_0_0
- added S1: JS102000SAQN, Switch:JS102000SAQN
- added TP1: TPB1,27, BeagleBone_Blue_R3:TPB1,27
- added TP2: LSP10, solpad:LSP10
- BT1: value 79523211 -> 79528211; device Battery Holder:79523211 -> Battery Holder:79528211
- R3: value (none) -> 100
- U1: device Microcontroller:ATTINY85-20PU -> Microcontroller:ATTINY85-20SU
Connections:
- removed net N$3: R3.1, SG1.-
- new net BEEP: TP1.TP, U1.PB4
- new net LED: R3.2, U1.PB1
- new net N$7: D2.A, R3.1
- net DET: now also Q1.COLLECTOR, U1.PB3; no longer SENS-1.P$1, U1.PB0
- net EMT: now also U1.PB2; no longer U1.PB1
- net GND: now also D1.C, D2.C, Q1.EMITTER, TP2.MP; no longer SENS-1.P$2, SENS-1.P$4, SG1.+
- net N$1: now also D1.A; no longer SENS-1.P$3
- net N$2: now also BT1.-, S1.1; no longer R3.2, U1.PB4
- net VCC: now also S1.2; no longer BT1.-
Other:
- moved on the sheet: BT1, R3
